File: HV_Charger.kicad_sch (KiCad schematic)
At the start: 21 parts

Commit message: Updated
Parts:
- added J?: Banana_Connector, symbol Connector_Generic:Conn_01x02
- added J?: AC Input, symbol Connector_Generic:Conn_01x02
- added R? (x2): 15K, symbol Device:R
Connections:
- new net: J?.2 (Pin_2), R?.1
- new net: J?.1 (Pin_1), R?.2
- new net: J?.1 (Pin_1), R?.1
- new net: J?.2 (Pin_2), R?.2
Changed lines of the file:
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@@
+    (stroke (width 0) (type default) (color 0 0 0 0))
+  )
+  (wire (pts (xy 58.42 163.83) (xy 67.31 163.83))
     (stroke (width 0) (type default) (color 0 0 0 0))
   )
@@
     (stroke (width 0) (type default) (color 0 0 0 0))
   )
+  (wire (pts (xy 41.91 161.29) (xy 50.8 161.29))
+    (stroke (width 0) (type default) (color 0 0 0 0))
+  )
   (polyline (pts (xy 59.69 53.34) (xy 132.08 53.34))
+    (stroke (width 0) (type default) (color 0 0 0 0))
+  )
+  (wire (pts (xy 41.91 163.83) (xy 50.8 163.83))
+    (stroke (width 0) (type default) (color 0 0 0 0))
+  )
+  (wire (pts (xy 58.42 161.29) (xy 67.31 161.29))
     (stroke (width 0) (type default) (color 0 0 0 0))
   )
@@
     (pin "9")
   )
+  (symbol (lib_id "Device:R") (at 54.61 163.83 270) (unit 1)
+    (in_bom yes) (on_board yes)
+    (property "Reference" "R?" (id 0) (at 54.61 166.37 90))
+    (property "Value" "15K" (id 1) (at 54.61 163.83 90))
+    (property "Footprint" "" (id 2) (at 54.61 162.052 90)
+      (effects (font (size 1.27 1.27)) hide)
+    )
+    (property "Datasheet" "~" (id 3) (at 54.61 163.83 0)
+      (effects (font (size 1.27 1.27)) hide)
+    )
+    (pin "1")
+    (pin "2")
+  )
   (symbol (lib_id "Device:LED") (at 108.585 28.575 180) (unit 1)
     (in_bom yes) (on_board yes)
@@
     (pin "2")
   )
+  (symbol (lib_id "Device:R") (at 54.61 161.29 270) (unit 1)
+    (in_bom yes) (on_board yes)
+    (property "Reference" "R?" (id 0) (at 54.61 159.385 90))
+    (property "Value" "15K" (id 1) (at 54.61 161.29 90))
+    (property "Footprint" "" (id 2) (at 54.61 159.512 90)
+      (effects (font (size 1.27 1.27)) hide)
+    )
+    (property "Datasheet" "~" (id 3) (at 54.61 161.29 0)
+      (effects (font (size 1.27 1.27)) hide)
+    )
+    (pin "1")
+    (pin "2")
+  )
   (symbol (lib_id "Jumper:Jumper_2_Bridged") (at 35.56 93.98 0) (unit 1)
     (in_bom yes) (on_board yes) (fields_autoplaced)
@@
     (pin "2")
   )
+  (symbol (lib_id "Connector_Generic:Conn_01x02") (at 72.39 161.29 0) (unit 1)
+    (in_bom yes) (on_board yes)
+    (property "Reference" "J?" (id 0) (at 71.12 155.575 0)
+      (effects (font (size 1.27 1.27)) (justify left))
+    )
+    (property "Value" "Banana_Connector" (id 1) (at 71.12 158.115 0)
+      (effects (font (size 1.27 1.27)) (justify left))
+    )
+    (property "Footprint" "" (id 2) (at 72.39 161.29 0)
+      (effects (font (size 1.27 1.27)) hide)
+    )
+    (property "Datasheet" "~" (id 3) (at 72.39 161.29 0)
+      (effects (font (size 1.27 1.27)) hide)
+    )
+    (pin "1")
+    (pin "2")
+  )
+  (symbol (lib_id "Connector_Generic:Conn_01x02") (at 36.83 163.83 180) (unit 1)
+    (in_bom yes) (on_board yes) (fields_autoplaced)
+    (property "Reference" "J?" (id 0) (at 36.83 154.94 0))
+    (property "Value" "AC Input" (id 1) (at 36.83 157.48 0))
+    (property "Footprint" "" (id 2) (at 36.83 163.83 0)
+      (effects (font (size 1.27 1.27)) hide)
+    )
+    (property "Datasheet" "~" (id 3) (at 36.83 163.83 0)
+      (effects (font (size 1.27 1.27)) hide)
+    )
+    (pin "1")
+    (pin "2")
+  )
   (symbol (lib_id "Connector_Generic:Conn_02x03_Odd_Even") (at 193.04 28.575 0) (unit 1)
     (in_bom yes) (on_board yes) (fields_autoplaced)
@@
       (reference "J?") (unit 1) (value "Expansion_Port") (footprint "")
     )
+    (path "/ebf5a38e-403a-4106-b6ce-4841dfc214c0"
+      (reference "J?") (unit 1) (value "Banana_Connector") (footprint "")
+    )
+    (path "/fc0c64c2-f56d-4589-bec0-9f436cccf30b"
+      (reference "J?") (unit 1) (value "AC Input") (footprint "")
+    )
     (path "/fd6efbf5-6a00-4931-ac7c-db6c727772c9"
       (reference "J?") (unit 1) (value "CAN Bridge") (footprint "")
@@
       (reference "R?") (unit 1) (value "IMD") (footprint "")
     )
+    (path "/2c366dc5-d43d-4e8d-b48c-960380cef255"
+      (reference "R?") (unit 1) (value "15K") (footprint "")
+    )
+    (path "/5ad18ff0-e076-452f-896f-da63b26e3683"
+      (reference "R?") (unit 1) (value "15K") (footprint "")
+    )
     (path "/910b9e07-7401-4d24-8508-f8c4f29a9270"
