File: HV_Charger.kicad_pcb (KiCad board)
At the start: 2 copper layers, 184.6 x 54.2 mm, 35 parts, among them J1 HVIL, J11 Conn_02x06_Top_Bottom, J13 3557-2, J2 E-Stop, J3 PP Connector, J4 IMD Indicator, J5 AMS Indicator, J6 CAN, J7 CAN_Expansion1, J8 CAN_Expansion2, J9 DC Input, Q1 Q_PMOS_SGD

Commit message: Done
Routing:
- added copper zone on F.Cu, net Net-(H1-Pad1)
- added copper zone on F.Cu, net Net-(H2-Pad1)
Changed lines of the file:
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@@
     (connect_pads yes (clearance 0.508))
     (min_thickness 0.254) (filled_areas_thickness no)
-    (fill (thermal_gap 0.508) (thermal_bridge_width 0.508))
+    (fill yes (thermal_gap 0.508) (thermal_bridge_width 0.508))
     (polygon
       (pts
@@
         (xy 84.2 70.6)
         (xy 132.4 70.6)
+      )
+    )
+  )
+  (zone (net 24) (net_name "Net-(H1-Pad1)") (layer "F.Cu") (hatch edge 0.508)
+    (connect_pads yes (clearance 0.508))
+    (min_thickness 0.254) (filled_areas_thickness no)
+    (fill yes (thermal_gap 0.508) (thermal_bridge_width 0.508))
+    (polygon
+      (pts
+        (xy 237.4 108.4)
+        (xy 224.6 108.4)
+        (xy 224.6 78)
+        (xy 237.4 78)
       )
     )
@@
       )
     )
+  )
+  (zone (net 25) (net_name "Net-(H2-Pad1)") (layer "F.Cu") (hatch edge 0.508)
+    (connect_pads yes (clearance 0.508))
+    (min_thickness 0.254) (filled_areas_thickness no)
+    (fill yes (thermal_gap 0.508) (thermal_bridge_width 0.508))
+    (polygon
+      (pts
+        (xy 222 78)
+        (xy 222 108.8)
+        (xy 209 108.8)
+        (xy 209.2 78)
+      )
+    )

Commit message: Made corrections
Parts:
- added R7: 100k, Resistor_SMD:R_0603_1608Metric, F.Cu at (87.8, 82.2)
- moved JP1 17.6 mm to (118.2, 76.7)
- moved JP2 17.6 mm to (121.3, 76.7)
- moved J3 17.6 mm to (119.6, 64.9)
- moved J2 12.6 mm to (135.2, 65.3)
- moved J9 5.98 mm to (225.6, 64.9), turned to 0 degrees
- moved J8 5.60 mm to (183.5, 64.8)
- moved JP3 5.25 mm to (167.9, 91.0)
- moved JP4 5.25 mm to (164.1, 91.0)
- moved R4 5.25 mm to (166.0, 84.6)
- moved J6 4.31 mm to (151.4, 65.3)
- moved R2 2.41 mm to (114.0, 79.6)
- moved H1 1.44 mm to (233.2, 106.4), turned to 90 degrees
- moved H2 1.08 mm to (216.4, 106.4), turned to 90 degrees
Routing:
- net 24V: track 199.7 -> 234.1 mm
- net AMS: track 0.00 -> 31.8 mm
- net CAN L: track 46.3 -> 76.9 mm
- net IMD: track 0.28 -> 26.0 mm
- net Net-(H2-Pad1): track 0.00 -> 25.2 mm
- net Net-(H1-Pad1): track 0.00 -> 25.1 mm
- net AMS_LO: track 0.00 -> 18.6 mm
- net Pilot_OUT: track 35.2 -> 52.9 mm
- net Prox_OUT: track 36.1 -> 52.7 mm
- net CAN H: track 42.9 -> 59.1 mm
- net Net-(J9-Pad1): track 0.00 -> 12.0 mm
- net Net-(J9-Pad2): track 0.00 -> 11.0 mm
- net IMD_LO: track 16.1 -> 25.2 mm
- net Shutdown_OUT: track 61.4 -> 55.6 mm
- net CAN L Bridge: track 22.1 -> 16.7 mm
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- added copper zone on B.Cu, net GND
- removed copper zone on F.Cu, net AMS
- removed copper zone on F.Cu, net AMS_LO
- removed copper zone on F.Cu, net IMD
- removed copper zone on F.Cu, net IMD_LO
- removed copper zone on F.Cu, net Net-(D3-Pad1)
- removed copper zone on F.Cu, net Net-(H1-Pad1)
- removed copper zone on F.Cu, net Net-(H2-Pad1)
- removed copper zone on F.Cu, net Net-(J9-Pad1)
- removed copper zone on F.Cu, net Net-(J9-Pad2)
Other:
- board text added: "High Voltage"
- board text added: "Low Voltage"
